File: pcb/SillyWilly58.kicad_pcb (KiCad board)
At the start: 2 copper layers, 142.5 x 106.3 mm, 83 parts, among them J1 LED, J2 4PIN, J3 OLED, P1 i2c_pin, P2 i2c_pin, SW1 SW_PUSH, SW10 SW_PUSH, SW11 SW_PUSH, SW12 SW_PUSH, SW13 SW_PUSH, SW14 SW_PUSH, SW15 SW_PUSH, SW16 SW_PUSH, SW17 SW_PUSH, SW18 SW_PUSH, SW19 SW_PUSH, SW2 SW_PUSH, SW20 SW_PUSH, SW21 SW_PUSH, SW22 SW_PUSH, SW23 SW_PUSH, SW24 SW_PUSH, SW25 SW_PUSH, SW26 SW_PUSH, SW27 SW_PUSH, SW28 SW_PUSH, SW29 SW_PUSH, SW3 SW_PUSH, SW4 SW_PUSH, SW5 SW_PUSH, SW6 SW_PUSH, SW7 SW_PUSH, SW8 SW_PUSH, SW9 SW_PUSH, U1 ProMicro

Commit message: Fixed some more trace stuff
Parts:
- D1, D10, D11, D12, D13, D14, D15, D16, D17, D18, D19, D2, D20, D21, D22, D23, D24, D25, D26, D27, D28, D29, D3, D4, D5, D6, D7, D8, D9: footprint Lily58-footprint:Diode_SOD123 -> SillyWilly58-footprint:Diode_SOD123
- J2: footprint Lily58-footprint:MJ-4PP-9 -> SillyWilly58-footprint:MJ-4PP-9
- SW1, SW10, SW11, SW12, SW13, SW14, SW15, SW16, SW17, SW18, SW19, SW2, SW20, SW21, SW22, SW23, SW24, SW25, SW26, SW27, SW28, SW29, SW3, SW4, SW5, SW6, SW7, SW8, SW9: footprint v2:KailhLowProfile_Hotswap_V2 -> SillyWilly58-footprint:KailhLowProfile_Hotswap_V2
- TH1, TH2: footprint Lily58-footprint:M2_HOLE_PCB -> SillyWilly58-footprint:M2_HOLE_PCB
Routing:
- net Net-(D28-Pad2): track 38.2 -> 34.0 mm
- net col4: track 275.5 -> 276.2 mm
Other:
- board text added: "Romans 3:23 Luke 13:3 Romans 10:9-10"
- board text added: "Romans 6:23 Titus 3:5 John 3:36"
