File: pcb/SillyWilly58.kicad_pcb (KiCad board)
At the start: 2 copper layers, 142.5 x 106.3 mm, 83 parts, among them J1 LED, J2 4PIN, J3 OLED, P1 i2c_pin, P2 i2c_pin, SW1 SW_PUSH, SW10 SW_PUSH, SW11 SW_PUSH, SW12 SW_PUSH, SW13 SW_PUSH, SW14 SW_PUSH, SW15 SW_PUSH, SW16 SW_PUSH, SW17 SW_PUSH, SW18 SW_PUSH, SW19 SW_PUSH, SW2 SW_PUSH, SW20 SW_PUSH, SW21 SW_PUSH, SW22 SW_PUSH, SW23 SW_PUSH, SW24 SW_PUSH, SW25 SW_PUSH, SW26 SW_PUSH, SW27 SW_PUSH, SW28 SW_PUSH, SW29 SW_PUSH, SW3 SW_PUSH, SW4 SW_PUSH, SW5 SW_PUSH, SW6 SW_PUSH, SW7 SW_PUSH, SW8 SW_PUSH, SW9 SW_PUSH, U1 ProMicro

Commit message: Created 3D model
Parts:
- removed TH1, TH2: HOLE, SillyWilly58-footprint:M2_HOLE_PCB
Changed lines of the file:
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@@
-		(embedded_fonts no)
-	)
-	(footprint "SillyWilly58-footprint:M2_HOLE_PCB"
-		(layer "F.Cu")
-		(at 86 85)
-		(property "Reference" "TH1"
-			(at 0 2.7 0)
-			(layer "F.SilkS")
-			(hide yes)
-			(effects
-				(font
-					(size 1 1)
-					(thickness 0.15)
-				)
-			)
-		)
-		(property "Value" "HOLE"
-			(at 0 -2.6 0)
-			(layer "F.Fab")
-			(effects
-				(font
-					(size 1 1)
-					(thickness 0.15)
-				)
-			)
-		)
-		(property "Datasheet" ""
-			(at 0 0 0)
-			(layer "F.Fab")
-			(hide yes)
-			(effects
-				(font
-					(size 1.27 1.27)
-				)
-			)
-		)
-		(property "Description" ""
-			(at 0 0 0)
-			(layer "F.Fab")
-			(hide yes)
-			(effects
-				(font
-					(size 1.27 1.27)
-				)
-			)
-		)
-		(attr through_hole)
-		(duplicate_pad_numbers_are_jumpers no)
-		(pad "" thru_hole circle
-			(at 0 0)
-			(size 4 4)
-			(drill 2.4)
-			(layers "*.Cu" "*.Mask")
-			(remove_unused_layers no)
-		)
-		(embedded_fonts no)
-	)
-	(footprint "SillyWilly58-footprint:M2_HOLE_PCB"
-		(layer "F.Cu")
-		(at 108 85)
-		(property "Reference" "TH2"
-			(at 0 2.7 0)
-			(layer "F.SilkS")
-			(hide yes)
-			(effects
-				(font
-					(size 1 1)
-					(thickness 0.15)
-				)
-			)
-		)
-		(property "Value" "HOLE"
-			(at 0 -2.6 0)
-			(layer "F.Fab")
-			(effects
-				(font
-					(size 1 1)
-					(thickness 0.15)
-				)
-			)
-		)
-		(property "Datasheet" ""
-			(at 0 0 0)
-			(layer "F.Fab")
-			(hide yes)
-			(effects
-				(font
-					(size 1.27 1.27)
-				)
-			)
-		)
-		(property "Description" ""
-			(at 0 0 0)
-			(layer "F.Fab")
-			(hide yes)
-			(effects
-				(font
-					(size 1.27 1.27)
-				)
-			)
-		)
-		(attr through_hole)
-		(duplicate_pad_numbers_are_jumpers no)
-		(pad "" thru_hole circle
-			(at 0 0)
-			(size 4 4)
-			(drill 2.4)
-			(layers "*.Cu" "*.Mask")
-			(remove_unused_layers no)
-		)
 		(embedded_fonts no)
 	)

Commit message: Removed some unneeded stuff
Parts:
- J1: footprint Lily58-footprint:LED -> SillyWilly58-footprint:LED
- J3: footprint Lily58-footprint:OLED_4Pin -> SillyWilly58-footprint:OLED_4Pin
- JP1, JP2, JP3, JP4, JP5, JP6, JP7, JP8: footprint Lily58-footprint:Jumper -> SillyWilly58-footprint:Jumper
- P1, P2: footprint Lily58-footprint:1pin_conn -> SillyWilly58-footprint:1pin_conn
- R1, R2: footprint Lily58-footprint:RESISTOR_mini -> SillyWilly58-footprint:RESISTOR_mini
- RSW1: footprint Lily58-footprint:TACT_SWITCH_TVBP06 -> SillyWilly58-footprint:TACT_SWITCH_TVBP06
- TH3, TH4, TH5, TH6, TH7: footprint Lily58-footprint:HOLE_M2_TH -> SillyWilly58-footprint:HOLE_M2_TH
- U1: footprint Lily58-footprint:ProMicro_rev2 -> SillyWilly58-footprint:ProMicro_rev2
- W1: footprint Lily58-footprint:jumper_data -> SillyWilly58-footprint:jumper_data
Changed lines of the file:
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@@
 		)
 	)
-	(footprint "Lily58-footprint:RESISTOR_mini"
+	(footprint "SillyWilly58-footprint:RESISTOR_mini"
 		(layer "F.Cu")
 		(at 84.688035 56.039272 -90)
@@
 		)
 	)
-	(footprint "Lily58-footprint:RESISTOR_mini"
+	(footprint "SillyWilly58-footprint:RESISTOR_mini"
 		(layer "F.Cu")
 		(at 86.938035 56.039272 -90)
@@
 		)
 	)
-	(footprint "Lily58-footprint:1pin_conn"
+	(footprint "SillyWilly58-footprint:1pin_conn"
 		(layer "F.Cu")
 		(at 84.7 60.7 180)
@@
 		)
 	)
-	(footprint "Lily58-footprint:1pin_conn"
+	(footprint "SillyWilly58-footprint:1pin_conn"
 		(layer "F.Cu")
 		(at 86.9 60.7 180)
@@
 		)
 	)
-	(footprint "Lily58-footprint:HOLE_M2_TH"
+	(footprint "SillyWilly58-footprint:HOLE_M2_TH"
 		(layer "F.Cu")
 		(at 129.6 59.6)
@@
 		(embedded_fonts no)
 	)
-	(footprint "Lily58-footprint:HOLE_M2_TH"
+	(footprint "SillyWilly58-footprint:HOLE_M2_TH"
 		(layer "F.Cu")
 		(at 205.8 61.8)
@@
 		(embedded_fonts no)
 	)
-	(footprint "Lily58-footprint:HOLE_M2_TH"
+	(footprint "SillyWilly58-footprint:HOLE_M2_TH"
 		(layer "F.Cu")
 		(at 129.6 97.6)
@@
 		(embedded_fonts no)
 	)
-	(footprint "Lily58-footprint:HOLE_M2_TH"
+	(footprint "SillyWilly58-footprint:HOLE_M2_TH"
 		(layer "F.Cu")
 		(at 205.8 100)
@@
 		(embedded_fonts no)
 	)
-	(footprint "Lily58-footprint:HOLE_M2_TH"
+	(footprint "SillyWilly58-footprint:HOLE_M2_TH"
 		(layer "F.Cu")
 		(at 105 114.8 90)
@@
 		(embedded_fonts no)
 	)
-	(footprint "Lily58-footprint:ProMicro_rev2"
+	(footprint "SillyWilly58-footprint:ProMicro_rev2"
 		(layer "F.Cu")
 		(at 101 56)
@@
 		(embedded_fonts no)
 	)
-	(footprint "Lily58-footprint:Jumper"
+	(footprint "SillyWilly58-footprint:Jumper"
 		(layer "F.Cu")
 		(at 104.3 69.3 90)
@@
 		)
 	)
-	(footprint "Lily58-footprint:Jumper"
+	(footprint "SillyWilly58-footprint:Jumper"
 		(layer "F.Cu")
 		(at 101.7 69.3 90)
@@
 		)
 	)
-	(footprint "Lily58-footprint:Jumper"
+	(footprint "SillyWilly58-footprint:Jumper"
 		(layer "F.Cu")
 		(at 99.2 69.3 90)
@@
 		)
 	)
-	(footprint "Lily58-footprint:TACT_SWITCH_TVBP06"
+	(footprint "SillyWilly58-footprint:TACT_SWITCH_TVBP06"
 		(layer "F.Cu")
 		(at 85 67.7 90)
@@
 		(embedded_fonts no)
 	)
-	(footprint "Lily58-footprint:jumper_data"
+	(footprint "SillyWilly58-footprint:jumper_data"
 		(layer "F.Cu")
 		(at 89 60.7 90)
@@
 		(embedded_fonts no)
 	)
-	(footprint "Lily58-footprint:Jumper"
+	(footprint "SillyWilly58-footprint:Jumper"
 		(layer "F.Cu")
 		(at 96.7 69.3 90)
@@
 		)
 	)
-	(footprint "Lily58-footprint:LED"
+	(footprint "SillyWilly58-footprint:LED"
 		(layer "F.Cu")
 		(at 112.7 81.1 180)
@@
 		(embedded_fonts no)
 	)
-	(footprint "Lily58-footprint:OLED_4Pin"
+	(footprint "SillyWilly58-footprint:OLED_4Pin"
 		(layer "F.Cu")
 		(at 96.7 74.6)
@@
 		(embedded_fonts no)
 	)
-	(footprint "Lily58-footprint:Jumper"
+	(footprint "SillyWilly58-footprint:Jumper"
 		(layer "B.Cu")
 		(at 101.7 69.3 90)
@@
 		)
 	)
-	(footprint "Lily58-footprint:Jumper"
+	(footprint "SillyWilly58-footprint:Jumper"
 		(layer "B.Cu")
 		(at 99.2 69.3 90)
@@
 		)
 	)
-	(footprint "Lily58-footprint:Jumper"
+	(footprint "SillyWilly58-footprint:Jumper"
 		(layer "B.Cu")
 		(at 96.7 69.3 90)
@@
 		)
 	)
-	(footprint "Lily58-footprint:Jumper"
+	(footprint "SillyWilly58-footprint:Jumper"
 		(layer "B.Cu")
 		(at 104.3 69.3 90)
